File: DCDC-FusePCB.kicad_sch (KiCad schematic)
At the start: 3 parts, among them J1 Conn_01x02_Socket, J2 Conn_01x02_Socket

Commit message: precharge board
Parts:
- added C1: 4.7uF, Capacitor_SMD:C_0805_2012Metric, symbol Device:C
- added D1, D2: LED, LED_SMD:LED_0805_2012Metric, symbol Device:LED
- added J3, J4, J6: Conn_01x02_Socket, Connector_Molex:Molex_Sabre_43160-0102_1x02_P7.49mm_Vertical, symbol Connector:Conn_01x02_Socket
- added J5: Precharge Resistor Breakout, Connector_Molex:Molex_Sabre_43160-0102_1x02_P7.49mm_Vertical, symbol Connector:Conn_01x02_Socket
- added R1, R2: 10k, Resistor_SMD:R_0805_2012Metric, symbol Device:R
- added R3: 100k, Resistor_SMD:R_0805_2012Metric, symbol Device:R
- added R4, R5: 22.1k, Resistor_SMD:R_0805_2012Metric, symbol Device:R
- added U1, U3: FDP3651U, footprints:TO-220-3_16P51X10P67_ONS, symbol 2025-06-07_04-14-49:FDP3651U
- added U2: TCMT1100, Package_SO:SOP-4_4.4x2.6mm_P1.27mm, symbol Isolator:TCMT1100
Connections:
- net at F1.1: now also J5.1 (Pin_1), U1.2 (D); no longer J2.2 (Pin_2)
- net HVin: now reaches F1.2, J1.2 (Pin_2)
- net GNDin: now reaches J1.1 (Pin_1), J2.1 (Pin_1)
- new net: J2.2 (Pin_2), J5.2 (Pin_2), U1.3 (S)
- new net: D2.2 (A), R5.2
- new net: R1.2, U2.2
- new net: D1.2 (A), R4.2
- new net +12Vsupp: J6.2 (Pin_2), U2.4
- new net DC/DC out: D2.1 (K), J4.2 (Pin_2), U3.2 (D)
- new net GNDout: C1.2, J3.1 (Pin_1), J4.1 (Pin_1), R1.1, R5.1
- new net GNDsupp: D1.1 (K), J6.1 (Pin_1), R2.2
- new net Gate_Drive: R2.1, R4.1, U1.1 (G), U2.3, U3.1 (G)
- new net LowPassIn: J3.2 (Pin_2), R3.1, U3.3 (S)
- new net LowPassOut: C1.1, R3.2, U2.1
Other:
- note added: "DC/DC output"
- note added: "Precharge Indicator"
- moved on the sheet: F1, J1, J2

Commit message: filled zones
Parts:
- added Q1: IPI200N15N3_G, TO254P457X1003X1598-3P, symbol IPI200N15N3_G:IPI200N15N3_G
Other:
- note added: "<- DC/DC input"
- note added: "DC/DC output after precharge ->"
Changed lines of the file:
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@@
+		)
+	)
+	(text "<- DC/DC input"
+		(exclude_from_sim no)
+		(at 244.856 51.308 0)
+		(effects
+			(font
+				(size 1.27 1.27)
+			)
+		)
+	)
+	(text "DC/DC output after precharge ->"
+		(exclude_from_sim no)
+		(at 245.618 80.264 0)
+		(effects
+			(font
+				(size 1.27 1.27)
+			)
 		)
 	)
@@
 					(unit 1)
 				)
+			)
+		)
+	)
+	(symbol
+		(lib_id "IPI200N15N3_G:IPI200N15N3_G")
+		(at 121.92 82.55 0)
+		(unit 1)
+		(exclude_from_sim no)
+		(in_bom yes)
+		(on_board yes)
+		(dnp no)
+		(fields_autoplaced yes)
+		(property "Reference" "Q1"
+			(at 133.35 78.7399 0)
+			(effects
+				(font
+					(size 1.27 1.27)
+				)
+				(justify left)
+			)
+		)
+		(property "Value" "IPI200N15N3_G"
+			(at 133.35 81.2799 0)
+			(effects
+				(font
+					(size 1.27 1.27)
+				)
+				(justify left)
+			)
+		)
+		(property "Footprint" "TO254P457X1003X1598-3P"
+			(at 133.35 181.28 0)
+			(effects
+				(font
+					(size 1.27 1.27)
+				)
+				(justify left top)
+				(hide yes)
+			)
+		)
+		(property "Datasheet" ""
+			(at 133.35 281.28 0)
+			(effects
+				(font
+					(size 1.27 1.27)
+				)
+				(justify left top)
+				(hide yes)
+			)
+		)
+		(property "Description" "MOSFET N-CH 150V 50A TO262-3"
+			(at 121.92 82.55 0)
+			(effects
+				(font
+					(size 1.27 1.27)
+				)
+				(hide yes)
+			)
+		)
+		(property "Height" "4.572"
+			(at 133.35 481.28 0)
+			(effects
+				(font
+					(size 1.27 1.27)
+				)
+				(justify left top)
+				(hide yes)
+			)
+		)
+		(property "Mouser Part Number" ""
+			(at 133.35 581.28 0)
+			(effects
+				(font
+					(size 1.27 1.27)
+				)
+				(justify left top)
+				(hide yes)
+			)
+		)
+		(property "Mouser Price/Stock" ""
+			(at 133.35 681.28 0)
+			(effects
+				(font
+					(size 1.27 1.27)
+				)
+				(justify left top)
+				(hide yes)
+			)
+		)
+		(property "Manufacturer_Name" "Infineon"
+			(at 133.35 781.28 0)
+			(effects
+				(font
+					(size 1.27 1.27)
+				)
+				(justify left top)
+				(hide yes)
+			)
+		)
+		(property "Manufacturer_Part_Number" "IPI200N15N3 G"
+			(at 133.35 881.28 0)
+			(effects
+				(font
+					(size 1.27 1.27)
+				)
+				(justify left top)
+				(hide yes)
+			)
+		)
+		(pin "1"
+		)
+		(pin "2"
+		)
+		(pin "3"
+		)
+		(instances
+			(project ""
+				(path "/15bce5be-1762-44e2-9cff-c5950a572cde"
+					(reference "Q1")
+					(unit 1)
+				)

Commit message: Changes
Parts:
- removed U1, U3: FDP3651U, footprints:TO-220-3_16P51X10P67_ONS, symbol 2025-06-07_04-14-49:FDP3651U
- added Q2: IPI200N15N3_G, footprints:TO-220-3_16P51X10P67_ONS, symbol IPI200N15N3_G:IPI200N15N3_G
- Q1: footprint TO254P457X1003X1598-3P -> footprints:TO-220-3_16P51X10P67_ONS
Connections:
- net DC/DC out: now also Q2.2 (D)
- net Gate_Drive: now also Q1.1 (G), Q2.1 (G)
- net LowPassIn: now also Q2.3 (S)
- net at F1.1, J5.1 (Pin_1): now also Q1.3 (S)
- net at J2.2 (Pin_2), J5.2 (Pin_2): now also Q1.2 (D)
Other:
- moved on the sheet: Q1
